File: meccano_micro.brd (EAGLE design)
At the start: 78.4 x 48.2 mm, 35 parts, among them U1 LM1117MP-3.3

Commit message: pin labels fix and added pinout documentation.
Changed pin labels “S(1,2,3,4)” to “D(01,02,03,04)”
Parts:
- renumbered S1 to D01, S2 to D02, S3 to D03, S4 to D04
Changed lines of the file:
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@@
 <?xml version="1.0" encoding="utf-8"?>
 <!DOCTYPE eagle SYSTEM "eagle.dtd">
-<eagle version="7.3.0">
+<eagle version="7.2.0">
 <drawing>
 <settings>
@@
 <attribute name="OC_FARNELL" value="176432" x="54.61" y="39.37" size="1.778" layer="27" display="off"/>
 </element>
-<element name="S1" library="wirepad" package="1,6/0,8" value="" x="8.89" y="36.83" smashed="yes" rot="R180">
+<element name="D01" library="wirepad" package="1,6/0,8" value="" x="8.89" y="36.83" smashed="yes" rot="R180">
 <attribute name="NAME" x="8.509" y="37.973" size="0.7" layer="25" ratio="10" rot="R90"/>
 <attribute name="VALUE" x="8.89" y="36.23" size="0.0254" layer="27" rot="R180"/>
 </element>
-<element name="S2" library="wirepad" package="1,6/0,8" value="" x="19.05" y="36.83" smashed="yes">
+<element name="D02" library="wirepad" package="1,6/0,8" value="" x="19.05" y="36.83" smashed="yes">
 <attribute name="NAME" x="18.669" y="37.973" size="0.7" layer="25" ratio="10" rot="R90"/>
 <attribute name="VALUE" x="19.05" y="37.43" size="0.0254" layer="27"/>
 </element>
-<element name="S3" library="wirepad" package="1,6/0,8" value="" x="30.48" y="36.83" smashed="yes">
+<element name="D03" library="wirepad" package="1,6/0,8" value="" x="30.48" y="36.83" smashed="yes">
 <attribute name="NAME" x="30.099" y="37.973" size="0.7" layer="25" ratio="10" rot="R90"/>
 <attribute name="VALUE" x="30.48" y="37.43" size="0.0254" layer="27"/>
 </element>
-<element name="S4" library="wirepad" package="1,6/0,8" value="" x="40.64" y="36.83" smashed="yes">
+<element name="D04" library="wirepad" package="1,6/0,8" value="" x="40.64" y="36.83" smashed="yes">
 <attribute name="NAME" x="40.259" y="37.973" size="0.7" layer="25" ratio="10" rot="R90"/>
 <attribute name="VALUE" x="40.64" y="37.43" size="0.0254" layer="27"/>
@@
 </signal>
 <signal name="HV1">
-<contactref element="S1" pad="1"/>
+<contactref element="D01" pad="1"/>
 <contactref element="HIGH" pad="1"/>
 <wire x1="9.25" y1="48.75" x2="11.25" y2="50.75" width="0.5" layer="1"/>
@@
 </signal>
 <signal name="HV2">
-<contactref element="S2" pad="1"/>
+<contactref element="D02" pad="1"/>
 <contactref element="HIGH" pad="2"/>
 <wire x1="13.75" y1="43.25" x2="13.75" y2="50.75" width="0.5" layer="1"/>
@@
 </signal>
 <signal name="HV3">
-<contactref element="S3" pad="1"/>
+<contactref element="D03" pad="1"/>
 <contactref element="HIGH" pad="5"/>
 <wire x1="21.75" y1="48.75" x2="21.75" y2="50.75" width="0.5" layer="1"/>
@@
 </signal>
 <signal name="HV4">
-<contactref element="S4" pad="1"/>
+<contactref element="D04" pad="1"/>
 <contactref element="HIGH" pad="6"/>
 <wire x1="35.5" y1="39.5" x2="24.25" y2="50.75" width="0.5" layer="1"/>

Commit message: Update board designer
Parts:
- C3: value 10uF -> 0.1uF
- renumbered D01 to S1, D02 to S2, D03 to S3, D04 to S4
Routing:
- net GND: track 0.00 -> 45.9 mm, vias 0 -> 1
- net N$4: track 47.2 -> 58.6 mm
- net LV4: track 56.1 -> 58.7 mm
Other:
- board text added: "(c) 2016 - Magazine Luiza LuizaLabs Meccano Micro - r.1.1"
- board text removed: "(c) 2015 - Magazine Luiza Arquitetura de Solucoes Meccano Micro - r.1.1"
Changed lines of the file:
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@@
 <?xml version="1.0" encoding="utf-8"?>
 <!DOCTYPE eagle SYSTEM "eagle.dtd">
-<eagle version="7.2.0">
+<eagle version="7.3.0">
 <drawing>
 <settings>
@@
 <layers>
 <layer number="1" name="Top" color="4" fill="1" visible="yes" active="yes"/>
-<layer number="16" name="Bottom" color="1" fill="1" visible="no" active="yes"/>
+<layer number="16" name="Bottom" color="1" fill="1" visible="yes" active="yes"/>
 <layer number="17" name="Pads" color="2" fill="1" visible="yes" active="yes"/>
 <layer number="18" name="Vias" color="2" fill="1" visible="yes" active="yes"/>
@@
 <circle x="74.93" y="34.29" radius="1.5" width="0" layer="20"/>
 <circle x="3.175" y="34.925" radius="1.5" width="0" layer="20"/>
-<text x="45.085" y="48.26" size="1.1" layer="25">(c) 2015 - Magazine Luiza
-Arquitetura de Solucoes
+<text x="45.085" y="48.26" size="1.1" layer="25">(c) 2016 - Magazine Luiza
+LuizaLabs
 Meccano Micro - r.1.1</text>
 <text x="11.43" y="58.42" size="0.8128" layer="25" rot="R270">LV4</text>
@@
 </autorouter>
 <elements>
-<element name="C3" library="capacitor-wima" package="C2.5-4" value="10uF" x="38.735" y="66.04" rot="R270"/>
+<element name="C3" library="capacitor-wima" package="C2.5-4" value="0.1uF" x="38.735" y="66.04" smashed="yes" rot="R270">
+<attribute name="NAME" x="40.894" y="67.691" size="1.27" layer="25" ratio="10" rot="R270"/>
+<attribute name="VALUE" x="35.306" y="67.691" size="0.8128" layer="27" ratio="10" rot="R270"/>
+</element>
 <element name="C4" library="rcl" package="B45181B" value="47uF" x="8.89" y="44.45" smashed="yes">
 <attribute name="NAME" x="5.969" y="47.244" size="1.27" layer="25" ratio="10"/>
@@
 <attribute name="OC_FARNELL" value="176432" x="54.61" y="39.37" size="1.778" layer="27" display="off"/>
 </element>
-<element name="D01" library="wirepad" package="1,6/0,8" value="" x="8.89" y="36.83" smashed="yes" rot="R180">
+<element name="S1" library="wirepad" package="1,6/0,8" value="" x="8.89" y="36.83" smashed="yes" rot="R180">
 <attribute name="NAME" x="8.509" y="37.973" size="0.7" layer="25" ratio="10" rot="R90"/>
 <attribute name="VALUE" x="8.89" y="36.23" size="0.0254" layer="27" rot="R180"/>
 </element>
-<element name="D02" library="wirepad" package="1,6/0,8" value="" x="19.05" y="36.83" smashed="yes">
+<element name="S2" library="wirepad" package="1,6/0,8" value="" x="19.05" y="36.83" smashed="yes">
 <attribute name="NAME" x="18.669" y="37.973" size="0.7" layer="25" ratio="10" rot="R90"/>
 <attribute name="VALUE" x="19.05" y="37.43" size="0.0254" layer="27"/>
 </element>
-<element name="D03" library="wirepad" package="1,6/0,8" value="" x="30.48" y="36.83" smashed="yes">
+<element name="S3" library="wirepad" package="1,6/0,8" value="" x="30.48" y="36.83" smashed="yes">
 <attribute name="NAME" x="30.099" y="37.973" size="0.7" layer="25" ratio="10" rot="R90"/>
 <attribute name="VALUE" x="30.48" y="37.43" size="0.0254" layer="27"/>
 </element>
-<element name="D04" library="wirepad" package="1,6/0,8" value="" x="40.64" y="36.83" smashed="yes">
+<element name="S4" library="wirepad" package="1,6/0,8" value="" x="40.64" y="36.83" smashed="yes">
 <attribute name="NAME" x="40.259" y="37.973" size="0.7" layer="25" ratio="10" rot="R90"/>
 <attribute name="VALUE" x="40.64" y="37.43" size="0.0254" layer="27"/>
@@
 </element>
 <element name="VCC-S1" library="wirepad" package="1,6/0,8" value="" x="6.35" y="36.83" smashed="yes">
-<attribute name="NAME" x="5.588" y="37.846" size="0.7" layer="25" ratio="10" rot="R90"/>
+<attribute name="NAME" x="6.223" y="37.846" size="0.7" layer="25" ratio="10" rot="R90"/>
 <attribute name="VALUE" x="6.35" y="37.43" size="0.0254" layer="27"/>
 </element>
@@
 <vertex x="0" y="31.75"/>
 </polygon>
-<wire x1="64.515" y1="57.64" x2="74.93" y2="66.04" width="0" layer="19" extent="1-1"/>
+<wire x1="74.93" y1="66.04" x2="76.2" y2="66.04" width="0.4064" layer="16"/>
+<wire x1="76.2" y1="66.04" x2="77.47" y2="64.77" width="0.4064" layer="16"/>
+<wire x1="77.47" y1="64.77" x2="77.47" y2="45.72" width="0.4064" layer="16"/>
+<wire x1="77.47" y1="45.72" x2="67.31" y2="35.56" width="0.4064" layer="16"/>
+<wire x1="67.31" y1="35.56" x2="59.69" y2="35.56" width="0.4064" layer="16"/>
+<wire x1="59.69" y1="35.56" x2="58.42" y2="36.83" width="0.4064" layer="16"/>
+<via x="61.595" y="67.31" extent="1-16" drill="0.6" shape="octagon"/>
 </signal>
 <signal name="5V">
@@
 <wire x1="51.25" y1="41.75" x2="51.3588" y2="41.6306" width="0.5" layer="1"/>
 <wire x1="61" y1="40.75" x2="66" y2="40.75" width="0.5" layer="1"/>
-<wire x1="61" y1="40.5" x2="61" y2="40.75" width="0.5" layer="1"/>
-<wire x1="59.75" y1="39.25" x2="61" y2="40.5" width="0.5" layer="1"/>
+<wire x1="59.73" y1="39.23" x2="61" y2="40.75" width="0.5" layer="1"/>
+<wire x1="59.75" y1="39.25" x2="59.73" y2="39.23" width="0.5" layer="1"/>
 <wire x1="51.75" y1="39.25" x2="59.75" y2="39.25" width="0.5" layer="1"/>
 <wire x1="51.25" y1="39.75" x2="51.75" y2="39.25" width="0.5" layer="1"/>
@@
 </signal>
 <signal name="HV1">
-<contactref element="D01" pad="1"/>
+<contactref element="S1" pad="1"/>
 <contactref element="HIGH" pad="1"/>
 <wire x1="9.25" y1="48.75" x2="11.25" y2="50.75" width="0.5" layer="1"/>
@@
 </signal>
 <signal name="HV2">
-<contactref element="D02" pad="1"/>
+<contactref element="S2" pad="1"/>
 <contactref element="HIGH" pad="2"/>
 <wire x1="13.75" y1="43.25" x2="13.75" y2="50.75" width="0.5" layer="1"/>
@@
 </signal>
 <signal name="HV3">
-<contactref element="D03" pad="1"/>
+<contactref element="S3" pad="1"/>
 <contactref element="HIGH" pad="5"/>
 <wire x1="21.75" y1="48.75" x2="21.75" y2="50.75" width="0.5" layer="1"/>
@@
 </signal>
 <signal name="HV4">
-<contactref element="D04" pad="1"/>
+<contactref element="S4" pad="1"/>
 <contactref element="HIGH" pad="6"/>
 <wire x1="35.5" y1="39.5" x2="24.25" y2="50.75" width="0.5" layer="1"/>
@@
 <wire x1="24.25" y1="61" x2="24.13" y2="60.96" width="0.5" layer="16"/>
 <wire x1="73" y1="58.25" x2="74.75" y2="58.25" width="0.5" layer="16"/>
-<wire x1="72" y1="57.25" x2="73" y2="58.25" width="0.5" layer="16"/>
-<wire x1="48.75" y1="57.25" x2="72" y2="57.25" width="0.5" layer="16"/>
-<wire x1="46.5" y1="59.5" x2="48.75" y2="57.25" width="0.5" layer="16"/>
+<wire x1="70.73" y1="54.71" x2="73" y2="58.25" width="0.5" layer="16"/>
+<wire x1="51.29" y1="54.71" x2="70.73" y2="54.71" width="0.5" layer="16"/>
+<wire x1="46.5" y1="59.5" x2="51.29" y2="54.71" width="0.5" layer="16"/>
 <wire x1="74.75" y1="58.25" x2="74.93" y2="58.42" width="0.5" layer="16"/>
 <wire x1="46.5" y1="59.5" x2="46.5" y2="59.75" width="0.5" layer="16"/>
@@
 <contactref element="SV1" pad="1"/>
 <wire x1="55" y1="67.75" x2="48.75" y2="67.75" width="0.5" layer="1"/>
-<wire x1="55" y1="47.71" x2="55" y2="67.75" width="0.5" layer="1"/>
-<wire x1="65.14" y1="47.73" x2="55" y2="47.71" width="0.5" layer="1"/>
+<wire x1="55" y1="40.09" x2="55" y2="67.75" width="0.5" layer="1"/>
+<wire x1="55" y1="40.09" x2="59.055" y2="40.005" width="0.5" layer="1"/>
+<wire x1="59.055" y1="40.005" x2="64.77" y2="47.095" width="0.5" layer="1"/>
+<wire x1="64.77" y1="47.095" x2="65.14" y2="47.73" width="0.5" layer="1"/>
 <wire x1="64.87" y1="48" x2="65.14" y2="47.73" width="0.5" layer="16"/>
 <wire x1="74.5" y1="48" x2="64.87" y2="48" width="0.5" layer="16"/>
@@
 </signal>
 </signals>
-<errors>
-</errors>
 </board>
 </drawing>

Commit message: Fix Configuration and Logical GPIO components
Parts:
- turned HIGH to 180 degrees
- turned LOW to 180 degrees
Connections:
- net 3V: no longer JP1.2
- net GND: now also JP1.2
Routing:
- net GND: track 45.9 -> 0.00 mm, vias 1 -> 0
- net LV1: track 101.2 -> 64.8 mm, vias 1 -> 2
- net 3V: track 133.9 -> 103.1 mm
- net HV1: track 15.1 -> 33.5 mm
- net HV3: track 17.7 -> 34.8 mm
- net HV4: track 23.6 -> 36.6 mm
- net LV3: track 64.6 -> 77.2 mm, vias 2 -> 1
- net 5V: track 162.3 -> 150.5 mm
- net LV4: track 58.7 -> 70.2 mm, vias 1 -> 2
- net N$4: track 58.6 -> 69.8 mm, vias 1 -> 0
- net LV2: track 67.4 -> 61.2 mm
- net N$7: track 84.9 -> 80.4 mm, vias 2 -> 0
- net HV2: track 16.5 -> 15.1 mm
- net N$11: track 37.4 -> 36.2 mm
- net N$6: track 30.4 -> 29.5 mm
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