File: meccano_micro.sch (EAGLE design)
At the start: 35 parts, among them U1 LM1117MP-3.3

Commit message: pin labels fix and added pinout documentation.
Changed pin labels “S(1,2,3,4)” to “D(01,02,03,04)”
Parts:
- renumbered S1 to D01, S2 to D02, S3 to D03, S4 to D04
Changed lines of the file:
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@@
 <?xml version="1.0" encoding="utf-8"?>
 <!DOCTYPE eagle SYSTEM "eagle.dtd">
-<eagle version="7.3.0">
+<eagle version="7.2.0">
 <drawing>
 <settings>
@@
 <part name="GND3" library="supply1" deviceset="GND" device=""/>
 <part name="VCC-S1" library="wirepad" deviceset="1,6/0,8" device=""/>
-<part name="S1" library="wirepad" deviceset="1,6/0,8" device=""/>
+<part name="D01" library="wirepad" deviceset="1,6/0,8" device=""/>
 <part name="GND-S1" library="wirepad" deviceset="1,6/0,8" device=""/>
 <part name="VCC-S2" library="wirepad" deviceset="1,6/0,8" device=""/>
-<part name="S2" library="wirepad" deviceset="1,6/0,8" device=""/>
+<part name="D02" library="wirepad" deviceset="1,6/0,8" device=""/>
 <part name="GND-S2" library="wirepad" deviceset="1,6/0,8" device=""/>
 <part name="5V2" library="supply1" deviceset="VCC" device="" value="5V"/>
@@
 <part name="LOW" library="con-lstb" deviceset="MA06-1" device=""/>
 <part name="VCC-S3" library="wirepad" deviceset="1,6/0,8" device=""/>
-<part name="S3" library="wirepad" deviceset="1,6/0,8" device=""/>
+<part name="D03" library="wirepad" deviceset="1,6/0,8" device=""/>
 <part name="GND-S3" library="wirepad" deviceset="1,6/0,8" device=""/>
 <part name="5V5" library="supply1" deviceset="VCC" device="" value="5V"/>
 <part name="GND10" library="supply1" deviceset="GND" device=""/>
 <part name="VCC-S4" library="wirepad" deviceset="1,6/0,8" device=""/>
-<part name="S4" library="wirepad" deviceset="1,6/0,8" device=""/>
+<part name="D04" library="wirepad" deviceset="1,6/0,8" device=""/>
 <part name="GND-S4" library="wirepad" deviceset="1,6/0,8" device=""/>
 <part name="5V6" library="supply1" deviceset="VCC" device="" value="5V"/>
@@
 <instance part="GND3" gate="1" x="88.9" y="27.94"/>
 <instance part="VCC-S1" gate="P" x="2.54" y="12.7" rot="R270"/>
-<instance part="S1" gate="P" x="10.16" y="12.7" rot="R270"/>
+<instance part="D01" gate="P" x="10.16" y="12.7" rot="R270"/>
 <instance part="GND-S1" gate="P" x="17.78" y="12.7" rot="R270"/>
 <instance part="VCC-S2" gate="P" x="40.64" y="12.7" rot="R270"/>
-<instance part="S2" gate="P" x="48.26" y="12.7" rot="R270"/>
+<instance part="D02" gate="P" x="48.26" y="12.7" rot="R270"/>
 <instance part="GND-S2" gate="P" x="55.88" y="12.7" rot="R270"/>
 <instance part="5V2" gate="VCC" x="2.54" y="0" rot="R180"/>
@@
 <instance part="LOW" gate="1" x="137.16" y="-38.1" rot="MR180"/>
 <instance part="VCC-S3" gate="P" x="187.96" y="15.24" rot="R270"/>
-<instance part="S3" gate="P" x="195.58" y="15.24" rot="R270"/>
+<instance part="D03" gate="P" x="195.58" y="15.24" rot="R270"/>
 <instance part="GND-S3" gate="P" x="203.2" y="15.24" rot="R270"/>
 <instance part="5V5" gate="VCC" x="187.96" y="2.54" rot="R180"/>
 <instance part="GND10" gate="1" x="203.2" y="5.08"/>
 <instance part="VCC-S4" gate="P" x="226.06" y="15.24" rot="R270"/>
-<instance part="S4" gate="P" x="233.68" y="15.24" rot="R270"/>
+<instance part="D04" gate="P" x="233.68" y="15.24" rot="R270"/>
 <instance part="GND-S4" gate="P" x="241.3" y="15.24" rot="R270"/>
 <instance part="5V6" gate="VCC" x="226.06" y="2.54" rot="R180"/>
@@
 <net name="HV1" class="0">
 <segment>
-<pinref part="S1" gate="P" pin="P"/>
+<pinref part="D01" gate="P" pin="P"/>
 <wire x1="10.16" y1="10.16" x2="10.16" y2="-30.48" width="0.1524" layer="91"/>
 <wire x1="10.16" y1="-30.48" x2="83.82" y2="-30.48" width="0.1524" layer="91"/>
@@
 <net name="HV2" class="0">
 <segment>
-<pinref part="S2" gate="P" pin="P"/>
+<pinref part="D02" gate="P" pin="P"/>
 <wire x1="48.26" y1="10.16" x2="48.26" y2="-33.02" width="0.1524" layer="91"/>
 <junction x="48.26" y="10.16"/>
@@
 <net name="HV3" class="0">
 <segment>
-<pinref part="S3" gate="P" pin="P"/>
+<pinref part="D03" gate="P" pin="P"/>
 <wire x1="195.58" y1="12.7" x2="195.58" y2="-53.34" width="0.1524" layer="91"/>
 <junction x="195.58" y="12.7"/>
@@
 <net name="HV4" class="0">
 <segment>
-<pinref part="S4" gate="P" pin="P"/>
+<pinref part="D04" gate="P" pin="P"/>
 <wire x1="233.68" y1="12.7" x2="233.68" y2="-55.88" width="0.1524" layer="91"/>
 <junction x="233.68" y="12.7"/>

Commit message: Update board designer
Parts:
- C3: value 10uF -> 0.1uF
- renumbered D01 to S1, D02 to S2, D03 to S3, D04 to S4
Changed lines of the file:
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@@
 <?xml version="1.0" encoding="utf-8"?>
 <!DOCTYPE eagle SYSTEM "eagle.dtd">
-<eagle version="7.2.0">
+<eagle version="7.3.0">
 <drawing>
 <settings>
@@
 <part name="GND3" library="supply1" deviceset="GND" device=""/>
 <part name="VCC-S1" library="wirepad" deviceset="1,6/0,8" device=""/>
-<part name="D01" library="wirepad" deviceset="1,6/0,8" device=""/>
+<part name="S1" library="wirepad" deviceset="1,6/0,8" device=""/>
 <part name="GND-S1" library="wirepad" deviceset="1,6/0,8" device=""/>
 <part name="VCC-S2" library="wirepad" deviceset="1,6/0,8" device=""/>
-<part name="D02" library="wirepad" deviceset="1,6/0,8" device=""/>
+<part name="S2" library="wirepad" deviceset="1,6/0,8" device=""/>
 <part name="GND-S2" library="wirepad" deviceset="1,6/0,8" device=""/>
 <part name="5V2" library="supply1" deviceset="VCC" device="" value="5V"/>
@@
 <part name="3V1" library="supply1" deviceset="VCC" device="" value="3V"/>
 <part name="3V2" library="supply1" deviceset="VCC" device="" value="3V"/>
-<part name="C3" library="capacitor-wima" deviceset="C" device="2.5/4" value="10uF"/>
+<part name="C3" library="capacitor-wima" deviceset="C" device="2.5/4" value="0.1uF"/>
 <part name="FTDI-GND" library="wirepad" deviceset="1,6/0,8" device=""/>
 <part name="FTDI-CTS" library="wirepad" deviceset="1,6/0,8" device=""/>
@@
 <part name="LOW" library="con-lstb" deviceset="MA06-1" device=""/>
 <part name="VCC-S3" library="wirepad" deviceset="1,6/0,8" device=""/>
-<part name="D03" library="wirepad" deviceset="1,6/0,8" device=""/>
+<part name="S3" library="wirepad" deviceset="1,6/0,8" device=""/>
 <part name="GND-S3" library="wirepad" deviceset="1,6/0,8" device=""/>
 <part name="5V5" library="supply1" deviceset="VCC" device="" value="5V"/>
 <part name="GND10" library="supply1" deviceset="GND" device=""/>
 <part name="VCC-S4" library="wirepad" deviceset="1,6/0,8" device=""/>
-<part name="D04" library="wirepad" deviceset="1,6/0,8" device=""/>
+<part name="S4" library="wirepad" deviceset="1,6/0,8" device=""/>
 <part name="GND-S4" library="wirepad" deviceset="1,6/0,8" device=""/>
 <part name="5V6" library="supply1" deviceset="VCC" device="" value="5V"/>
@@
 <instance part="GND3" gate="1" x="88.9" y="27.94"/>
 <instance part="VCC-S1" gate="P" x="2.54" y="12.7" rot="R270"/>
-<instance part="D01" gate="P" x="10.16" y="12.7" rot="R270"/>
+<instance part="S1" gate="P" x="10.16" y="12.7" rot="R270"/>
 <instance part="GND-S1" gate="P" x="17.78" y="12.7" rot="R270"/>
 <instance part="VCC-S2" gate="P" x="40.64" y="12.7" rot="R270"/>
-<instance part="D02" gate="P" x="48.26" y="12.7" rot="R270"/>
+<instance part="S2" gate="P" x="48.26" y="12.7" rot="R270"/>
 <instance part="GND-S2" gate="P" x="55.88" y="12.7" rot="R270"/>
 <instance part="5V2" gate="VCC" x="2.54" y="0" rot="R180"/>
@@
 <instance part="LOW" gate="1" x="137.16" y="-38.1" rot="MR180"/>
 <instance part="VCC-S3" gate="P" x="187.96" y="15.24" rot="R270"/>
-<instance part="D03" gate="P" x="195.58" y="15.24" rot="R270"/>
+<instance part="S3" gate="P" x="195.58" y="15.24" rot="R270"/>
 <instance part="GND-S3" gate="P" x="203.2" y="15.24" rot="R270"/>
 <instance part="5V5" gate="VCC" x="187.96" y="2.54" rot="R180"/>
 <instance part="GND10" gate="1" x="203.2" y="5.08"/>
 <instance part="VCC-S4" gate="P" x="226.06" y="15.24" rot="R270"/>
-<instance part="D04" gate="P" x="233.68" y="15.24" rot="R270"/>
+<instance part="S4" gate="P" x="233.68" y="15.24" rot="R270"/>
 <instance part="GND-S4" gate="P" x="241.3" y="15.24" rot="R270"/>
 <instance part="5V6" gate="VCC" x="226.06" y="2.54" rot="R180"/>
@@
 <net name="HV1" class="0">
 <segment>
-<pinref part="D01" gate="P" pin="P"/>
+<pinref part="S1" gate="P" pin="P"/>
 <wire x1="10.16" y1="10.16" x2="10.16" y2="-30.48" width="0.1524" layer="91"/>
 <wire x1="10.16" y1="-30.48" x2="83.82" y2="-30.48" width="0.1524" layer="91"/>
@@
 <net name="HV2" class="0">
 <segment>
-<pinref part="D02" gate="P" pin="P"/>
+<pinref part="S2" gate="P" pin="P"/>
 <wire x1="48.26" y1="10.16" x2="48.26" y2="-33.02" width="0.1524" layer="91"/>
 <junction x="48.26" y="10.16"/>
@@
 <net name="HV3" class="0">
 <segment>
-<pinref part="D03" gate="P" pin="P"/>
+<pinref part="S3" gate="P" pin="P"/>
 <wire x1="195.58" y1="12.7" x2="195.58" y2="-53.34" width="0.1524" layer="91"/>
 <junction x="195.58" y="12.7"/>
@@
 <net name="HV4" class="0">
 <segment>
-<pinref part="D04" gate="P" pin="P"/>
+<pinref part="S4" gate="P" pin="P"/>
 <wire x1="233.68" y1="12.7" x2="233.68" y2="-55.88" width="0.1524" layer="91"/>
 <junction x="233.68" y="12.7"/>

Commit message: Fix Configuration and Logical GPIO components
Connections:
- net 3V: no longer JP1.2
- net GND: now also JP1.2
Changed lines of the file:
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@@
 <part name="GND5" library="supply1" deviceset="GND" device=""/>
 <part name="3V1" library="supply1" deviceset="VCC" device="" value="3V"/>
-<part name="3V2" library="supply1" deviceset="VCC" device="" value="3V"/>
 <part name="C3" library="capacitor-wima" deviceset="C" device="2.5/4" value="0.1uF"/>
 <part name="FTDI-GND" library="wirepad" deviceset="1,6/0,8" device=""/>
@@
 <part name="5V7" library="supply1" deviceset="VCC" device="" value="5V"/>
 <part name="GND12" library="supply1" deviceset="GND" device=""/>
+<part name="GND13" library="supply1" deviceset="GND" device=""/>
 </parts>
 <sheets>
@@
 <instance part="GND5" gate="1" x="55.88" y="2.54"/>
 <instance part="3V1" gate="VCC" x="144.78" y="35.56" rot="R270"/>
-<instance part="3V2" gate="VCC" x="68.58" y="55.88"/>
 <instance part="C3" gate="G$1" x="111.76" y="12.7" rot="R90"/>
 <instance part="FTDI-GND" gate="P" x="96.52" y="96.52" rot="R270"/>
@@
 <instance part="5V7" gate="VCC" x="177.8" y="73.66"/>
 <instance part="GND12" gate="1" x="182.626" y="76.2" rot="R180"/>
+<instance part="GND13" gate="1" x="68.58" y="55.88" rot="R180"/>
 </instances>
 <busses>
@@
 <label x="210.82" y="73.66" size="1.778" layer="95"/>
 </segment>
+<segment>
+<wire x1="68.58" y1="50.8" x2="68.58" y2="53.34" width="0.1524" layer="91"/>
+<pinref part="JP1" gate="A" pin="2"/>
+<junction x="68.58" y="50.8"/>
+<pinref part="GND13" gate="1" pin="GND"/>
+</segment>
 </net>
 <net name="5V" class="0">
@@
 </segment>
 <segment>
-<pinref part="3V2" gate="VCC" pin="VCC"/>
-<wire x1="68.58" y1="50.8" x2="68.58" y2="53.34" width="0.1524" layer="91"/>
-<pinref part="JP1" gate="A" pin="2"/>
-<junction x="68.58" y="50.8"/>
-</segment>
-<segment>
